File: MATE ROV Float.kicad_pcb (KiCad board)
At the start: 2 copper layers, 60 x 50.2 mm, 54 parts, among them J1 Conn_02x02_Counter_Clockwise, J2 Conn_01x03, J3 Conn_01x02, J4 Conn_01x03, J5 AVR-ISP-6, J6 Conn_02x02_Counter_Clockwise, M1 Motor_DC, Q1 BSS138, Q2 BSS138, SW1 SW_Push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

Commit message: Add files via upload
Parts:
- moved D2 9.00 mm to (200.2, 82.0)
- moved R7 9.00 mm to (200.2, 79.0)
- moved D1 3.01 mm to (200.5, 88.0)
- moved R6 3.01 mm to (200.3, 85.0)
- moved C12 1.75 mm to (160.0, 85.2)
- moved C13 1.75 mm to (160.0, 82.5)
- moved C14 1.75 mm to (160.0, 79.8)
- moved J3 1.75 mm to (157.5, 74.2)
- moved R5 1.50 mm to (177.5, 76.5)
- moved REF** 1.50 mm to (201.8, 74.8)
- moved SW1 1.50 mm to (171.0, 74.8)
- moved U5 1.50 mm to (190.2, 85.2)
- moved REF** 1.25 mm to (149.8, 74.8)
- moved U3 1.00 mm to (166.5, 82.2)
Routing:
- net GND: track 10.1 -> 7.38 mm, vias 113 -> 106
- net Net-(U5-PIO[11]): track 27.9 -> 25.7 mm
- net VCC: track 115.4 -> 113.3 mm
- net Net-(J1-Pin_3): track 27.9 -> 26.3 mm
- net Net-(J1-Pin_4): track 30.7 -> 29.2 mm
- net Net-(U5-PIO[8]): track 2.61 -> 3.48 mm
- net (no net): vias 1 -> 0
Other:
- board size 60 x 50.2 mm -> 60 x 48.2 mm
