File: MATE ROV Float.kicad_sch (KiCad schematic)
At the start: 35 parts, among them J2 Conn_01x03, J3 Conn_01x02, J4 Conn_01x03, J5 AVR-ISP-6, J6 Conn_02x02_Counter_Clockwise, M1 Motor_DC, U1 ATmega328P-M, U2 AZ1117-5.0, U3 AZ1117-3.3, U4 DRV8220DRLR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

Commit message: Add files via upload
Connections:
- no-connect marks 0 -> 10
Changed lines of the file:
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@@
   (junction (at 217.17 130.81) (diameter 0) (color 0 0 0 0)
   )
+  (no_connect (at 60.96 65.405))
+  (no_connect (at 91.44 106.045))
+  (no_connect (at 91.44 88.265))
+  (no_connect (at 91.44 116.205))
+  (no_connect (at 91.44 113.665))
+  (no_connect (at 91.44 85.725))
+  (no_connect (at 91.44 108.585))
+  (no_connect (at 91.44 57.785))
+  (no_connect (at 91.44 111.125))
+  (no_connect (at 60.96 62.865))
   (wire (pts (xy 123.19 67.945) (xy 126.365 67.945))
     (stroke (width 0) (type default))
