File: communication.kicad_sch (KiCad schematic)
At the start: 16 parts, among them J1 Conn_02x02_Counter_Clockwise, Q1 BSS138, Q2 BSS138, SW1 SW_Push, U5 HC-05

Commit message: Add files via upload
Connections:
- no-connect marks 0 -> 23
Other:
- note added: "NEEDS CHECKING"
Changed lines of the file:
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@@
   (junction (at 100.965 69.215) (diameter 0) (color 0 0 0 0)
   )
+  (no_connect (at 116.84 100.33))
+  (no_connect (at 157.48 85.09))
+  (no_connect (at 157.48 110.49))
+  (no_connect (at 116.84 107.95))
+  (no_connect (at 116.84 82.55))
+  (no_connect (at 116.84 92.71))
+  (no_connect (at 116.84 95.25))
+  (no_connect (at 157.48 87.63))
+  (no_connect (at 157.48 100.33))
+  (no_connect (at 157.48 80.01))
+  (no_connect (at 157.48 90.17))
+  (no_connect (at 157.48 118.11))
+  (no_connect (at 157.48 92.71))
+  (no_connect (at 116.84 102.87))
+  (no_connect (at 116.84 74.93))
+  (no_connect (at 157.48 82.55))
+  (no_connect (at 116.84 87.63))
+  (no_connect (at 157.48 115.57))
+  (no_connect (at 116.84 115.57))
+  (no_connect (at 157.48 107.95))
+  (no_connect (at 116.84 105.41))
+  (no_connect (at 116.84 113.03))
+  (no_connect (at 157.48 77.47))
   (wire (pts (xy 109.22 88.9) (xy 109.22 85.09))
     (stroke (width 0) (type default))
@@
     (stroke (width 0) (type default))
   )
+  (text "NEEDS CHECKING\n" (at 165.735 75.565 0)
+    (effects (font (size 3 3)) (justify left bottom))
+  )
   (label "RX3.3v" (at 106.68 69.215 0) (fields_autoplaced)
